File: schematics/plug_controller/plug_controller.kicad_pcb (KiCad board)
At the start: 2 copper layers, 55.9 x 41.9 mm, 20 parts, among them J1 Conn_01x04, J2 Conn_01x01, J3 Conn_01x01, J4 Conn_01x01, J5 Conn_01x01, Q1 MMBT3904L, Q2 MMBT3904L, Q3 MMBT3904L, Q4 MMBT3904L, U1 MOC3063M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

Commit message: update footprints as assembling first design.
The triac pins were reversed.
The fuse footprints were not the holders i have.
The resistor between optotriac and triac should be larger.
Parts:
- D1, D2: value T25 -> Q_TRIAC_T25
- F1: footprint Fuse_Holders_and_Fuses:Fuseholder5x20_horiz_open_inline_Type-I -> Fuse_Holders_and_Fuses:Fuseholder5x20_horiz_open_lateral_Type-II
- R5, R6: value 300 -> 1K
- moved J5 27.0 mm to (181.9, 118.4), turned to 180 degrees
- moved F1 3.68 mm to (208.2, 88.9)
Connections:
- D2 pad 1: Net-(D1-Pad1) -> Net-(D2-Pad1)
- D2 pad 2: Net-(D2-Pad2) -> Net-(D1-Pad2)
- F1 pad 2: Net-(D1-Pad1) -> Net-(D1-Pad2)
- J3 pad 1: Net-(D1-Pad2) -> Net-(D1-Pad1)
- J4 pad 1: Net-(D2-Pad2) -> Net-(D2-Pad1)
- U1 pad 6: Net-(D1-Pad1) -> Net-(D1-Pad2)
- U2 pad 6: Net-(D1-Pad1) -> Net-(D1-Pad2)
Routing:
- net Net-(D1-Pad2): track 24.6 -> 60.8 mm, vias 0 -> 2
- net Net-(D2-Pad2): track 26.1 -> 0.00 mm
- net Net-(D2-Pad1): track 0.00 -> 24.4 mm, vias 0 -> 1
- net Net-(D1-Pad1): track 44.9 -> 24.4 mm, vias 2 -> 1
- net Net-(F1-Pad1): track 17.0 -> 35.5 mm
- removed copper zone on B.Cu, net Net-(F1-Pad1)
Other:
- outline, holes or cut-outs redrawn
